File: project.kicad_sch (KiCad schematic)
At the start: 160 parts, among them SW1 SW_Push, U1 ATmega32U4-A, Y1 16MHz

Commit message: halfway through leds
Parts:
- added C10, C11, C12, C13, C14, C15, C16, C17, C18, C19, C20, C21, C8: C_Small, symbol Device:C_Small
- added C9: (no value), symbol Device:C_Small
- added D10, D12, D13, D14, D15, D16, D17, D18, D19, D20, D21, D22, D23: WS2812B, LED_SMD:LED_WS2812B_PLCC4_5.0x5.0mm_P3.2mm, symbol LED:WS2812B
- added D11: (no value), symbol LED:WS2812B
Connections:
- net +5V: now also C10.1, C11.1, C12.1, C13.1, C14.1, C15.1, C16.1, C17.1, C18.1, C19.1, C20.1, C21.1, C8.1, C9.1, D10.1 (VDD), D11.1 (VDD), D12.1 (VDD), D13.1 (VDD), D14.1 (VDD), D15.1 (VDD), D16.1 (VDD), D17.1 (VDD), D18.1 (VDD), D19.1 (VDD), D20.1 (VDD), D21.1 (VDD), D22.1 (VDD), D23.1 (VDD)
- net COL0: now also U1.41 (PF0)
- net COL1: now also U1.40 (PF1)
- net COL10: now also U1.28 (PB4)
- net COL11: now also U1.27 (PD7)
- net COL12: now also U1.26 (PD6)
- net COL13: now also U1.25 (PD4)
- net COL14: now also U1.22 (PD5)
- net COL2: now also U1.39 (PF4)
- net COL3: now also U1.38 (PF5)
- net COL4: now also U1.37 (PF6)
- net COL5: now also U1.36 (PF7)
- net COL6: now also U1.32 (PC7)
- net COL7: now also U1.31 (PC6)
- net COL8: now also U1.30 (PB6)
- net COL9: now also U1.29 (PB5)
- net GND: now also C10.2, C11.2, C12.2, C13.2, C14.2, C15.2, C16.2, C17.2, C18.2, C19.2, C20.2, C21.2, C8.2, C9.2, D10.3 (VSS), D11.3 (VSS), D12.3 (VSS), D13.3 (VSS), D14.3 (VSS), D15.3 (VSS), D16.3 (VSS), D17.3 (VSS), D18.3 (VSS), D19.3 (VSS), D20.3 (VSS), D21.3 (VSS), D22.3 (VSS), D23.3 (VSS)
- net ROW0: now also U1.11 (PB3)
- net ROW1: now also U1.18 (PD0)
- net ROW2: now also U1.19 (PD1)
- net ROW3: now also U1.20 (PD2)
- net ROW4: now also U1.21 (PD3)
- net RGB LED: now reaches U1.10 (PB2)
- net RGB LED: now also D11.4 (DIN)
- new net: D21.2 (DOUT), D23.4 (DIN)
- new net: D19.2 (DOUT), D21.4 (DIN)
- new net: D20.2 (DOUT), D22.4 (DIN)
- new net: D18.2 (DOUT), D20.4 (DIN)
- new net: D17.2 (DOUT), D19.4 (DIN)
- new net: D13.2 (DOUT), D15.4 (DIN)
- new net: D11.2 (DOUT), D13.4 (DIN)
- new net: D15.2 (DOUT), D17.4 (DIN)
- new net: D10.2 (DOUT), D12.4 (DIN)
- new net: D10.4 (DIN), D23.2 (DOUT)
- new net: D16.2 (DOUT), D18.4 (DIN)
- new net: D12.2 (DOUT), D14.4 (DIN)
- new net: D14.2 (DOUT), D16.4 (DIN)
