File: project.kicad_pcb (KiCad board)
At the start: 2 copper layers, 160 parts, among them SW1 SW_Push, U1 ATmega32U4-A, Y1 16MHz

Commit message: halfway through leds
Parts:
- added C10: C_Small, Capacitor_SMD:C_0603_1608Metric, F.Cu at (48.5, -67.3)
- added C11: C_Small, Capacitor_SMD:C_0603_1608Metric, F.Cu at (10.3, -45.6)
- added C12: C_Small, Capacitor_SMD:C_0603_1608Metric, F.Cu at (37.2, -66.2)
- added C13: C_Small, Capacitor_SMD:C_0603_1608Metric, F.Cu at (21.0, -45.2)
- added C14: C_Small, Capacitor_SMD:C_0603_1608Metric, B.Cu at (216.7, -92.1)
- added C15: C_Small, Capacitor_SMD:C_0603_1608Metric, F.Cu at (32.8, -44.6)
- added C16: C_Small, Capacitor_SMD:C_0603_1608Metric, B.Cu at (178.6, -92.1)
- added C17: C_Small, Capacitor_SMD:C_0603_1608Metric, F.Cu at (47.6, -44.7)
- added C18: C_Small, Capacitor_SMD:C_0603_1608Metric, B.Cu at (140.5, -92.1)
- added C19: C_Small, Capacitor_SMD:C_0603_1608Metric, F.Cu at (60.2, -44.2)
- added C20: C_Small, Capacitor_SMD:C_0603_1608Metric, B.Cu at (111.9, -92.1)
- added C21: C_Small, Capacitor_SMD:C_0603_1608Metric, F.Cu at (72.6, -45.0)
- added C8: C_Small, Capacitor_SMD:C_0603_1608Metric, F.Cu at (60.2, -66.4)
- added C9: C_Small, Capacitor_SMD:C_0603_1608Metric, F.Cu at (0.00, -44.6)
- added D10: WS2812B, LED_SMD:LED_WS2812B_PLCC4_5.0x5.0mm_P3.2mm, F.Cu at (65.4, -60.7)
- added D11: WS2812B, LED_SMD:LED_WS2812B_PLCC4_5.0x5.0mm_P3.2mm, F.Cu at (-6.10, -51.6)
- added D12: WS2812B, LED_SMD:LED_WS2812B_PLCC4_5.0x5.0mm_P3.2mm, F.Cu at (54.2, -60.6)
- added D13: WS2812B, LED_SMD:LED_WS2812B_PLCC4_5.0x5.0mm_P3.2mm, F.Cu at (4.70, -52.5)
- added D14: WS2812B, LED_SMD:LED_WS2812B_PLCC4_5.0x5.0mm_P3.2mm, F.Cu at (42.0, -60.8)
- added D15: WS2812B, LED_SMD:LED_WS2812B_PLCC4_5.0x5.0mm_P3.2mm, F.Cu at (16.4, -51.3)
- added D16: WS2812B, LED_SMD:LED_WS2812B_PLCC4_5.0x5.0mm_P3.2mm, B.Cu at (222.2, -92.1)
- added D17: WS2812B, LED_SMD:LED_WS2812B_PLCC4_5.0x5.0mm_P3.2mm, F.Cu at (26.0, -50.9)
- added D18: WS2812B, LED_SMD:LED_WS2812B_PLCC4_5.0x5.0mm_P3.2mm, B.Cu at (184.2, -92.1)
- added D19: WS2812B, LED_SMD:LED_WS2812B_PLCC4_5.0x5.0mm_P3.2mm, F.Cu at (38.9, -50.8)
- added D20: WS2812B, LED_SMD:LED_WS2812B_PLCC4_5.0x5.0mm_P3.2mm, B.Cu at (146.1, -92.1)
- added D21: WS2812B, LED_SMD:LED_WS2812B_PLCC4_5.0x5.0mm_P3.2mm, F.Cu at (54.6, -51.2)
- added D22: WS2812B, LED_SMD:LED_WS2812B_PLCC4_5.0x5.0mm_P3.2mm, B.Cu at (117.5, -92.1)
- added D23: WS2812B, LED_SMD:LED_WS2812B_PLCC4_5.0x5.0mm_P3.2mm, F.Cu at (65.0, -50.7)
Connections:
- net GND renamed e
- U1 pad 10: unconnected-(U1-Pad10) -> RGB LED

Commit message: stop here for discontinued rgb
Parts:
- C10, C11, C12, C13, C15, C17, C19, C21, C8, C9, D10, D11, D12, D13, D14, D15, D17, D19, D21, D23: moved to B.Cu
- moved D23 264.6 mm to (329.4, -39.7), turned to 180 degrees
- moved D10 263.5 mm to (327.0, -92.1), turned to 180 degrees
- moved C8 262.5 mm to (321.5, -92.1), turned to -90 degrees
- moved C21 262.4 mm to (335.0, -39.7), turned to -90 degrees
- moved D12 246.2 mm to (298.4, -92.1), turned to 180 degrees
- moved C10 245.6 mm to (292.9, -92.1), turned to -90 degrees
- moved D21 235.4 mm to (289.7, -39.7), turned to 180 degrees
- moved C19 235.1 mm to (295.3, -39.7), turned to -90 degrees
- moved D19 231.3 mm to (269.9, -39.7), turned to 180 degrees
- moved C17 227.9 mm to (275.4, -39.7), turned to -90 degrees
- moved D14 220.5 mm to (260.4, -92.1), turned to 180 degrees
- moved C12 219.1 mm to (254.8, -92.1), turned to -90 degrees
- moved D17 196.5 mm to (222.2, -39.7), turned to 180 degrees
- moved C15 195.1 mm to (227.8, -39.7), turned to -90 degrees
- moved C13 159.3 mm to (180.2, -39.7), turned to -90 degrees
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
Commit message: Please add screw holes, solenoid, and fill zones
Routing:
- net e: track 198.7 -> 739.6 mm, vias 2 -> 18
- net +5V: track 145.9 -> 680.8 mm, vias 5 -> 8
- net Net-(D10-Pad4): track 0.00 -> 80.6 mm, vias 0 -> 2
- net RGB LED: track 0.00 -> 52.7 mm, vias 0 -> 2
- net Net-(D18-Pad2): track 0.00 -> 50.3 mm, vias 0 -> 4
- net Net-(D16-Pad2): track 0.00 -> 50.3 mm, vias 0 -> 4
- net Net-(D14-Pad2): track 0.00 -> 50.3 mm, vias 0 -> 4
- net Net-(D12-Pad2): track 0.00 -> 50.3 mm, vias 0 -> 4
- net Net-(D17-Pad2): track 0.00 -> 44.1 mm
- net Net-(D15-Pad2): track 0.00 -> 44.1 mm
- net Net-(D20-Pad2): track 0.00 -> 42.3 mm, vias 0 -> 4
- net Net-(D21-Pad2): track 0.00 -> 36.1 mm
- net Net-(D11-Pad2): track 0.00 -> 36.1 mm
- net Net-(D10-Pad2): track 0.00 -> 34.8 mm, vias 0 -> 2
- net Net-(D19-Pad2): track 0.00 -> 16.3 mm
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